File: mainboard-v05/Avionics.kicad_sch (KiCad schematic)
At the start: 39 parts, among them J10 Conn_01x04, J15 Conn_01x02, J8 Conn_01x09, J9 Conn_01x03, U1 MAX706RESA, U2 ATSAMD51J19A-AU, U3 BMX160, Y1 32.768kHz

Commit message: Added more fields to BOM.
Parts:
- C3, C5, C7, C9, C? (x2): LCSC (none) -> C1591
- C? (x2): LCSC (none) -> C1691
- C? (x4): LCSC (none) -> C1592
- C? (x2): LCSC (none) -> C346204
- J10: LCSC (none) -> C780062
- J8: LCSC (none) -> C2883929
- J9: LCSC (none) -> C2883760
- L?: LCSC (none) -> C88173
- R1: LCSC (none) -> C844550
- R2: LCSC (none) -> C137807
- R3, R4, R44, R45: LCSC (none) -> C1511834
- R6: LCSC (none) -> C844773
Changed lines of the file:
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@@
       (effects (font (size 1.27 1.27)) hide)
     )
-    (property "LCSC" "" (at 256.54 139.7 0)
+    (property "LCSC" "C1591" (at 256.54 139.7 0)
       (effects (font (size 1.27 1.27)) hide)
     )
@@
       (effects (font (size 1.27 1.27)) hide)
     )
-    (property "LCSC" "" (at 152.4 87.63 0)
+    (property "LCSC" "C1691" (at 152.4 87.63 0)
       (effects (font (size 1.27 1.27)) hide)
     )
@@
       (effects (font (size 1.27 1.27)) hide)
     )
-    (property "LCSC" "" (at 147.32 87.63 0)
+    (property "LCSC" "C1592" (at 147.32 87.63 0)
       (effects (font (size 1.27 1.27)) hide)
     )
@@
       (effects (font (size 1.27 1.27)) hide)
     )
-    (property "LCSC" "" (at 142.24 87.63 0)
+    (property "LCSC" "C1592" (at 142.24 87.63 0)
       (effects (font (size 1.27 1.27)) hide)
     )
@@
       (effects (font (size 1.27 1.27)) hide)
     )
-    (property "LCSC" "" (at 66.04 87.63 0)
+    (property "LCSC" "C1592" (at 66.04 87.63 0)
       (effects (font (size 1.27 1.27)) hide)
     )
@@
       (effects (font (size 1.27 1.27)) hide)
     )
-    (property "LCSC" "" (at 137.16 97.79 0)
+    (property "LCSC" "C1592" (at 137.16 97.79 0)
       (effects (font (size 1.27 1.27)) hide)
     )
@@
       (effects (font (size 1.27 1.27)) hide)
     )
-    (property "LCSC" "" (at 128.27 100.33 0)
+    (property "LCSC" "C88173" (at 128.27 100.33 0)
       (effects (font (size 1.27 1.27)) hide)
     )
@@
       (effects (font (size 1.27 1.27)) hide)
     )
-    (property "LCSC" "" (at 142.24 97.79 0)
+    (property "LCSC" "C1691" (at 142.24 97.79 0)
       (effects (font (size 1.27 1.27)) hide)
     )
@@
       (effects (font (size 1.27 1.27)) hide)
     )
-    (property "LCSC" "" (at 41.91 105.41 0)
+    (property "LCSC" "C346204" (at 41.91 105.41 0)
       (effects (font (size 1.27 1.27)) hide)
     )
@@
       (effects (font (size 1.27 1.27)) hide)
     )
-    (property "LCSC" "" (at 41.91 113.03 0)
+    (property "LCSC" "C346204" (at 41.91 113.03 0)
       (effects (font (size 1.27 1.27)) hide)
     )
@@
       (effects (font (size 1.27 1.27)) hide)
     )
-    (property "LCSC" "" (at 55.88 123.19 0)
+    (property "LCSC" "C844550" (at 55.88 123.19 0)
       (effects (font (size 1.27 1.27)) hide)
     )
@@
       (effects (font (size 1.27 1.27)) hide)
     )
-    (property "LCSC" "" (at 81.28 81.28 0)
+    (property "LCSC" "C1511834" (at 81.28 81.28 0)
       (effects (font (size 1.27 1.27)) hide)
     )
@@
       (effects (font (size 1.27 1.27)) hide)
     )
-    (property "LCSC" "" (at 76.2 81.28 0)
+    (property "LCSC" "C1511834" (at 76.2 81.28 0)
       (effects (font (size 1.27 1.27)) hide)
     )
@@
       (effects (font (size 1.27 1.27)) hide)
     )
-    (property "LCSC" "" (at 55.88 130.81 0)
+    (property "LCSC" "C137807" (at 55.88 130.81 0)
       (effects (font (size 1.27 1.27)) hide)
     )
@@
       (effects (font (size 1.27 1.27)) hide)
     )
-    (property "LCSC" "" (at 137.16 87.63 0)
+    (property "LCSC" "C1591" (at 137.16 87.63 0)
       (effects (font (size 1.27 1.27)) hide)
     )
@@
       (effects (font (size 1.27 1.27)) hide)
     )
-    (property "LCSC" "" (at 60.96 132.08 0)
+    (property "LCSC" "C1591" (at 60.96 132.08 0)
       (effects (font (size 1.27 1.27)) hide)
     )
@@
       (effects (font (size 1.27 1.27)) hide)
     )
-    (property "LCSC" "" (at 233.68 53.34 0)
+    (property "LCSC" "C2883929" (at 233.68 53.34 0)
       (effects (font (size 1.27 1.27)) hide)
     )
@@
       (effects (font (size 1.27 1.27)) hide)
     )
-    (property "LCSC" "" (at 132.08 87.63 0)
+    (property "LCSC" "C1591" (at 132.08 87.63 0)
       (effects (font (size 1.27 1.27)) hide)
     )
@@
       (effects (font (size 1.27 1.27)) hide)
     )
-    (property "LCSC" "" (at 144.78 134.62 0)
+    (property "LCSC" "C1511834" (at 144.78 134.62 0)
       (effects (font (size 1.27 1.27)) hide)
     )
@@
       (effects (font (size 1.27 1.27)) hide)
     )
-    (property "LCSC" "" (at 157.48 137.16 0)
+    (property "LCSC" "C1511834" (at 157.48 137.16 0)
       (effects (font (size 1.27 1.27)) hide)
     )
@@
       (effects (font (size 1.27 1.27)) hide)
     )
-    (property "LCSC" "" (at 43.18 160.02 0)
+    (property "LCSC" "C1591" (at 43.18 160.02 0)
       (effects (font (size 1.27 1.27)) hide)
     )
@@
       (effects (font (size 1.27 1.27)) hide)
     )
-    (property "LCSC" "" (at 233.68 74.93 0)
+    (property "LCSC" "C2883760" (at 233.68 74.93 0)
       (effects (font (size 1.27 1.27)) hide)
     )
@@
       (effects (font (size 1.27 1.27)) hide)
     )
-    (property "LCSC" "" (at 233.68 90.17 0)
+    (property "LCSC" "C780062" (at 233.68 90.17 0)
       (effects (font (size 1.27 1.27)) hide)
     )
@@
       (effects (font (size 1.27 1.27)) hide)
     )
-    (property "LCSC" "" (at 214.63 132.08 0)
+    (property "LCSC" "C1591" (at 214.63 132.08 0)
       (effects (font (size 1.27 1.27)) hide)
     )
@@
       (effects (font (size 1.27 1.27)) hide)
     )
-    (property "LCSC" "" (at 85.09 123.19 0)
-      (effects (font (size 1.27 1.27)) hide)
-    )
+    (property "LCSC" "C844773" (at 85.09 123.19 0)
+      (effects (font (size 1.27 1.27)) hide)
+    )

Commit message: edits
Parts:
- U1: LCSC (none) -> C28380
- U2: LCSC (none) -> C619214
- U3: LCSC (none) -> C2655104
- Y1: LCSC (none) -> C32346
- gave numbers to parts that had none: 12

Commit message: Improved Py-Cubed BOM
Parts:
- D1, J15: LCSC (none) -> NotAvailable
- R41, R42, R7: LCSC (none) -> C1511834
Changed lines of the file:
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@@
       (effects (font (size 1.27 1.27)) hide)
     )
-    (property "LCSC" "" (at 52.07 54.61 0)
+    (property "LCSC" "C1511834" (at 52.07 54.61 0)
       (effects (font (size 1.27 1.27)) hide)
     )
@@
       (effects (font (size 1.27 1.27)) hide)
     )
-    (property "LCSC" "" (at 57.15 158.75 0)
+    (property "LCSC" "NotAvailable" (at 57.15 158.75 0)
       (effects (font (size 1.27 1.27)) hide)
     )
@@
       (effects (font (size 1.27 1.27)) hide)
     )
-    (property "LCSC" "" (at 255.27 127 0)
+    (property "LCSC" "C1511834" (at 255.27 127 0)
       (effects (font (size 1.27 1.27)) hide)
     )
@@
       (effects (font (size 1.27 1.27)) hide)
     )
-    (property "LCSC" "" (at 257.81 72.39 0)
+    (property "LCSC" "NotAvailable" (at 257.81 72.39 0)
       (effects (font (size 1.27 1.27)) hide)
     )
@@
       (effects (font (size 1.27 1.27)) hide)
     )
-    (property "LCSC" "" (at 76.2 168.91 0)
-      (effects (font (size 1.27 1.27)) hide)
-    )
+    (property "LCSC" "C1511834" (at 76.2 168.91 0)
+      (effects (font (size 1.27 1.27)) hide)
+    )
