File: mainboard-v05/Burn_Wires.kicad_sch (KiCad schematic)
At the start: 22 parts, among them Q20 NDS8434, Q21 NDS8434, Q4 IRLML2803, Q5 IRLML2803, Q6 MMBT2222AT, U16 PE014006

Commit message: Added more fields to BOM.
Parts:
- D4: LCSC (none) -> C5380706
- Q4, Q5: LCSC (none) -> C2590
- Q6: LCSC (none) -> C190608
- R32, R33: LCSC (none) -> C844773
Changed lines of the file:
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@@
       (effects (font (size 1.27 1.27)) hide)
     )
-    (property "LCSC" "" (at 157.48 57.15 0)
+    (property "LCSC" "C844773" (at 157.48 57.15 0)
       (effects (font (size 1.27 1.27)) hide)
     )
@@
       (effects (font (size 1.27 1.27)) hide)
     )
-    (property "LCSC" "" (at 58.42 35.56 0)
+    (property "LCSC" "C5380706" (at 58.42 35.56 0)
       (effects (font (size 1.27 1.27)) hide)
     )
@@
       (effects (font (size 1.27 1.27)) hide)
     )
-    (property "LCSC" "" (at 58.42 43.18 0)
+    (property "LCSC" "C190608" (at 58.42 43.18 0)
       (effects (font (size 1.27 1.27)) hide)
     )
@@
       (effects (font (size 1.27 1.27)) hide)
     )
-    (property "LCSC" "" (at 165.1 64.77 0)
+    (property "LCSC" "C2590" (at 165.1 64.77 0)
       (effects (font (size 1.27 1.27)) hide)
     )
@@
       (effects (font (size 1.27 1.27)) hide)
     )
-    (property "LCSC" "" (at 157.48 33.02 0)
+    (property "LCSC" "C844773" (at 157.48 33.02 0)
       (effects (font (size 1.27 1.27)) hide)
     )
@@
       (effects (font (size 1.27 1.27)) hide)
     )
-    (property "LCSC" "" (at 165.1 40.64 0)
-      (effects (font (size 1.27 1.27)) hide)
-    )
+    (property "LCSC" "C2590" (at 165.1 40.64 0)
+      (effects (font (size 1.27 1.27)) hide)
+    )

Commit message: edits
Parts:
- U16: LCSC (none) -> NotAvailable
Changed lines of the file:
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@@
     (effects (font (size 1.651 1.651)) (justify left bottom))
   )
-  (label "VBURN_A_IN" (at 124.46 30.48 180)
+  (label "VBURN_A_IN" (at 124.46 30.48 180) (fields_autoplaced)
     (effects (font (size 1.27 1.27)) (justify right bottom))
   )
-  (label "VBURN1" (at 213.36 35.56 180)
+  (label "VBURN1" (at 213.36 35.56 180) (fields_autoplaced)
     (effects (font (size 1.27 1.27)) (justify right bottom))
   )
-  (label "VBURN2" (at 213.36 59.69 180)
+  (label "VBURN2" (at 213.36 59.69 180) (fields_autoplaced)
     (effects (font (size 1.27 1.27)) (justify right bottom))
   )
@@
           (reference "#GND061") (unit 1)
         )
-        (path "/e3ac22ea-6806-4807-a025-571315789c25"
-          (reference "#GND?") (unit 1)
-        )
       )
     )
@@
           (reference "JP12") (unit 1)
         )
-        (path "/e3ac22ea-6806-4807-a025-571315789c25"
-          (reference "JP?") (unit 1)
-        )
       )
     )
@@
           (reference "R33") (unit 1)
         )
-        (path "/e3ac22ea-6806-4807-a025-571315789c25"
-          (reference "R?") (unit 1)
-        )
       )
     )
@@
           (reference "JP9") (unit 1)
         )
-        (path "/e3ac22ea-6806-4807-a025-571315789c25"
-          (reference "JP?") (unit 1)
-        )
       )
     )
@@
           (reference "D4") (unit 1)
         )
-        (path "/e3ac22ea-6806-4807-a025-571315789c25"
-          (reference "D?") (unit 1)
-        )
       )
     )
@@
         (path "/e3ac22ea-6806-4807-a025-571315789c25/00000000-0000-0000-0000-00005cec6476"
           (reference "#GND051") (unit 1)
-        )
-        (path "/e3ac22ea-6806-4807-a025-571315789c25"
-          (reference "#GND?") (unit 1)
         )
       )
@@
           (reference "R25") (unit 1)
         )
-        (path "/e3ac22ea-6806-4807-a025-571315789c25"
-          (reference "R?") (unit 1)
-        )
       )
     )
@@
           (reference "JP14") (unit 1)
         )
-        (path "/e3ac22ea-6806-4807-a025-571315789c25"
-          (reference "JP?") (unit 1)
-        )
       )
     )
@@
           (reference "#GND048") (unit 1)
         )
-        (path "/e3ac22ea-6806-4807-a025-571315789c25"
-          (reference "#GND?") (unit 1)
-        )
       )
     )
@@
           (reference "#GND056") (unit 1)
         )
-        (path "/e3ac22ea-6806-4807-a025-571315789c25"
-          (reference "#GND?") (unit 1)
-        )
       )
     )
@@
         (path "/e3ac22ea-6806-4807-a025-571315789c25/00000000-0000-0000-0000-00005cec6476"
           (reference "#GND064") (unit 1)
-        )
-        (path "/e3ac22ea-6806-4807-a025-571315789c25"
-          (reference "#GND?") (unit 1)
         )
       )
@@
           (reference "JP10") (unit 1)
         )
-        (path "/e3ac22ea-6806-4807-a025-571315789c25"
-          (reference "JP?") (unit 1)
-        )
       )
     )
@@
         (path "/e3ac22ea-6806-4807-a025-571315789c25/00000000-0000-0000-0000-00005cec6476"
           (reference "R28") (unit 1)
-        )
-        (path "/e3ac22ea-6806-4807-a025-571315789c25"
-          (reference "R?") (unit 1)
         )
       )
@@
           (reference "Q20") (unit 1)
         )
-        (path "/e3ac22ea-6806-4807-a025-571315789c25/00000000-0000-0000-0000-00005cec5a72"
-          (reference "U?") (unit 1)
-        )
       )
     )
@@
           (reference "Q21") (unit 1)
         )
-        (path "/e3ac22ea-6806-4807-a025-571315789c25/00000000-0000-0000-0000-00005cec5a72"
-          (reference "U?") (unit 1)
-        )
       )
     )
@@
           (reference "R27") (unit 1)
         )
-        (path "/e3ac22ea-6806-4807-a025-571315789c25"
-          (reference "R?") (unit 1)
-        )
       )
     )
@@
         (path "/e3ac22ea-6806-4807-a025-571315789c25/00000000-0000-0000-0000-00005cec6476"
           (reference "#GND054") (unit 1)
-        )
-        (path "/e3ac22ea-6806-4807-a025-571315789c25"
-          (reference "#GND?") (unit 1)
         )
       )
@@
           (reference "Q5") (unit 1)
         )
-        (path "/e3ac22ea-6806-4807-a025-571315789c25"
-          (reference "Q?") (unit 1)
-        )
       )
     )
@@
           (reference "R32") (unit 1)
         )
-        (path "/e3ac22ea-6806-4807-a025-571315789c25"
-          (reference "R?") (unit 1)
-        )
       )
     )
@@
           (reference "R37") (unit 1)
         )
-        (path "/e3ac22ea-6806-4807-a025-571315789c25"
-          (reference "R?") (unit 1)
-        )
       )
     )
@@
           (reference "JP11") (unit 1)
         )
-        (path "/e3ac22ea-6806-4807-a025-571315789c25"
-          (reference "JP?") (unit 1)
-        )
       )
     )
@@
         (path "/e3ac22ea-6806-4807-a025-571315789c25/00000000-0000-0000-0000-00005cec6476"
           (reference "#GND063") (unit 1)
-        )
-        (path "/e3ac22ea-6806-4807-a025-571315789c25"
-          (reference "#GND?") (unit 1)
         )
       )
@@
           (reference "R38") (unit 1)
         )
-        (path "/e3ac22ea-6806-4807-a025-571315789c25"
-          (reference "R?") (unit 1)
-        )
       )
     )
@@
           (reference "JP15") (unit 1)
         )
-        (path "/e3ac22ea-6806-4807-a025-571315789c25"
-          (reference "JP?") (unit 1)
-        )
       )
     )
@@
           (reference "JP13") (unit 1)
         )
-        (path "/e3ac22ea-6806-4807-a025-571315789c25"
-          (reference "JP?") (unit 1)
-        )
       )
     )
@@
           (reference "#GND062") (unit 1)
         )
-        (path "/e3ac22ea-6806-4807-a025-571315789c25"
-          (reference "#GND?") (unit 1)
-        )
       )
     )
@@
         (path "/e3ac22ea-6806-4807-a025-571315789c25/00000000-0000-0000-0000-00005cec6476"
           (reference "#GND052") (unit 1)
-        )
-        (path "/e3ac22ea-6806-4807-a025-571315789c25"
-          (reference "#GND?") (unit 1)
         )
       )
@@
       (effects (font (size 1.27 1.27)) hide)
     )
-    (property "LCSC" "" (at 81.28 33.02 0)
+    (property "LCSC" "NotAvailable" (at 81.28 33.02 0)
       (effects (font (size 1.27 1.27)) hide)
     )
@@
           (reference "U16") (unit 1)
         )
-        (path "/e3ac22ea-6806-4807-a025-571315789c25"
-          (reference "U?") (unit 1)
-        )
       )
     )
@@
           (reference "Q4") (unit 1)
         )
-        (path "/e3ac22ea-6806-4807-a025-571315789c25"
-          (reference "Q?") (unit 1)
-        )
       )
     )
@@
           (reference "#GND055") (unit 1)
         )
-        (path "/e3ac22ea-6806-4807-a025-571315789c25"
-          (reference "#GND?") (unit 1)
-        )
       )
     )
@@
           (reference "#GND060") (unit 1)
         )
-        (path "/e3ac22ea-6806-4807-a025-571315789c25"
-          (reference "#GND?") (unit 1)
-        )
       )
     )
@@
         (path "/e3ac22ea-6806-4807-a025-571315789c25/00000000-0000-0000-0000-00005cec6476"
           (reference "#GND049") (unit 1)
-        )
-        (path "/e3ac22ea-6806-4807-a025-571315789c25"
-          (reference "#GND?") (unit 1)
         )
       )
@@
           (reference "JP8") (unit 1)
         )
-        (path "/e3ac22ea-6806-4807-a025-571315789c25"
-          (reference "JP?") (unit 1)
-        )
-      )
+      )

Commit message: Improved Py-Cubed BOM
Parts:
- JP10, JP11, JP12, JP13, JP14, JP15, JP8, JP9, Q20, Q21: LCSC (none) -> NotAvailable
- R25, R27, R28: LCSC (none) -> C1511834
- R37, R38: LCSC (none) -> C5369222
Changed lines of the file:
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@@
       (effects (font (size 1.27 1.27)) hide)
     )
-    (property "LCSC" "" (at 215.9 67.31 0)
+    (property "LCSC" "NotAvailable" (at 215.9 67.31 0)
       (effects (font (size 1.27 1.27)) hide)
     )
@@
       (effects (font (size 1.27 1.27)) hide)
     )
-    (property "LCSC" "" (at 80.01 105.41 0)
+    (property "LCSC" "NotAvailable" (at 80.01 105.41 0)
       (effects (font (size 1.27 1.27)) hide)
     )
@@
       (effects (font (size 1.27 1.27)) hide)
     )
-    (property "LCSC" "" (at 50.8 48.26 0)
+    (property "LCSC" "C1511834" (at 50.8 48.26 0)
       (effects (font (size 1.27 1.27)) hide)
     )
@@
       (effects (font (size 1.27 1.27)) hide)
     )
-    (property "LCSC" "" (at 82.55 134.62 0)
+    (property "LCSC" "NotAvailable" (at 82.55 134.62 0)
       (effects (font (size 1.27 1.27)) hide)
     )
@@
       (effects (font (size 1.27 1.27)) hide)
     )
-    (property "LCSC" "" (at 125.73 105.41 0)
+    (property "LCSC" "NotAvailable" (at 125.73 105.41 0)
       (effects (font (size 1.27 1.27)) hide)
     )
@@
       (effects (font (size 1.27 1.27)) hide)
     )
-    (property "LCSC" "" (at 152.4 62.23 0)
+    (property "LCSC" "C1511834" (at 152.4 62.23 0)
       (effects (font (size 1.27 1.27)) hide)
     )
@@
       (effects (font (size 1.27 1.27)) (justify left bottom) hide)
     )
-    (property "LCSC" "" (at 190.5 38.1 0)
+    (property "LCSC" "NotAvailable" (at 190.5 38.1 0)
       (effects (font (size 1.27 1.27)) hide)
     )
@@
       (effects (font (size 1.27 1.27)) hide)
     )
-    (property "LCSC" "" (at 190.5 62.23 0)
+    (property "LCSC" "NotAvailable" (at 190.5 62.23 0)
       (effects (font (size 1.27 1.27)) hide)
     )
@@
       (effects (font (size 1.27 1.27)) hide)
     )
-    (property "LCSC" "" (at 152.4 38.1 0)
+    (property "LCSC" "C1511834" (at 152.4 38.1 0)
       (effects (font (size 1.27 1.27)) hide)
     )
@@
       (effects (font (size 1.27 1.27)) hide)
     )
-    (property "LCSC" "" (at 170.18 35.56 0)
+    (property "LCSC" "C5369222" (at 170.18 35.56 0)
       (effects (font (size 1.27 1.27)) hide)
     )
@@
       (effects (font (size 1.27 1.27)) hide)
     )
-    (property "LCSC" "" (at 215.9 43.18 0)
+    (property "LCSC" "NotAvailable" (at 215.9 43.18 0)
       (effects (font (size 1.27 1.27)) hide)
     )
@@
       (effects (font (size 1.27 1.27)) hide)
     )
-    (property "LCSC" "" (at 170.18 59.69 0)
+    (property "LCSC" "C5369222" (at 170.18 59.69 0)
       (effects (font (size 1.27 1.27)) hide)
     )
@@
       (effects (font (size 1.27 1.27)) hide)
     )
-    (property "LCSC" "" (at 128.27 134.62 0)
+    (property "LCSC" "NotAvailable" (at 128.27 134.62 0)
       (effects (font (size 1.27 1.27)) hide)
     )
@@
       (effects (font (size 1.27 1.27)) hide)
     )
-    (property "LCSC" "" (at 43.18 133.35 0)
+    (property "LCSC" "NotAvailable" (at 43.18 133.35 0)
       (effects (font (size 1.27 1.27)) hide)
     )
@@
       (effects (font (size 1.27 1.27)) hide)
     )
-    (property "LCSC" "" (at 39.37 105.41 0)
-      (effects (font (size 1.27 1.27)) hide)
-    )
+    (property "LCSC" "NotAvailable" (at 39.37 105.41 0)
+      (effects (font (size 1.27 1.27)) hide)
+    )
