File: mainboard-v05/Bus_Protection.kicad_sch (KiCad schematic)
At the start: 53 parts, among them Q11 MMDT2907, Q12 BSS138DWQ-7, Q13 BSS138DWQ-7, Q15 MBT2222ADW1T1, Q16 MBT2222ADW1T1, Q17 MMBT2907, Q18 BSS138DWQ-7, Q19 BSS138DWQ-7, Q7 MBT2222ADW1T1, Q8 MBT2222ADW1T1

Commit message: Added more fields to BOM.
Parts:
- C40, C41, C42, C8: LCSC (none) -> C1589
- Q11: LCSC (none) -> C414226
- Q12, Q13, Q18, Q19: LCSC (none) -> C3280240
- Q15, Q16, Q7, Q8: LCSC (none) -> C559075
- Q17: LCSC (none) -> C2914421
- R60, R92: LCSC (none) -> C844773
- R61, R62, R66, R67, R82, R83, R84, R85: LCSC (none) -> C1511834
Changed lines of the file:
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@@
       (effects (font (size 1.27 1.27)) hide)
     )
-    (property "LCSC" "" (at 29.21 68.58 0)
+    (property "LCSC" "C3280240" (at 29.21 68.58 0)
       (effects (font (size 1.27 1.27)) hide)
     )
@@
       (effects (font (size 1.27 1.27)) hide)
     )
-    (property "LCSC" "" (at 44.45 73.66 0)
+    (property "LCSC" "C3280240" (at 44.45 73.66 0)
       (effects (font (size 1.27 1.27)) hide)
     )
@@
       (effects (font (size 1.27 1.27)) hide)
     )
-    (property "LCSC" "" (at 45.72 58.42 0)
+    (property "LCSC" "C559075" (at 45.72 58.42 0)
       (effects (font (size 1.27 1.27)) hide)
     )
@@
       (effects (font (size 1.27 1.27)) hide)
     )
-    (property "LCSC" "" (at 45.72 40.64 0)
+    (property "LCSC" "C559075" (at 45.72 40.64 0)
       (effects (font (size 1.27 1.27)) hide)
     )
@@
       (effects (font (size 1.27 1.27)) hide)
     )
-    (property "LCSC" "" (at 50.8 77.47 0)
+    (property "LCSC" "C1589" (at 50.8 77.47 0)
       (effects (font (size 1.27 1.27)) hide)
     )
@@
       (effects (font (size 1.27 1.27)) hide)
     )
-    (property "LCSC" "" (at 50.8 38.1 0)
+    (property "LCSC" "C1511834" (at 50.8 38.1 0)
       (effects (font (size 1.27 1.27)) hide)
     )
@@
       (effects (font (size 1.27 1.27)) hide)
     )
-    (property "LCSC" "" (at 45.72 31.75 0)
+    (property "LCSC" "C1511834" (at 45.72 31.75 0)
       (effects (font (size 1.27 1.27)) hide)
     )
@@
       (effects (font (size 1.27 1.27)) hide)
     )
-    (property "LCSC" "" (at 87.63 58.42 0)
+    (property "LCSC" "C559075" (at 87.63 58.42 0)
       (effects (font (size 1.27 1.27)) hide)
     )
@@
       (effects (font (size 1.27 1.27)) hide)
     )
-    (property "LCSC" "" (at 87.63 40.64 0)
+    (property "LCSC" "C559075" (at 87.63 40.64 0)
       (effects (font (size 1.27 1.27)) hide)
     )
@@
       (effects (font (size 1.27 1.27)) hide)
     )
-    (property "LCSC" "" (at 92.71 77.47 0)
+    (property "LCSC" "C1589" (at 92.71 77.47 0)
       (effects (font (size 1.27 1.27)) hide)
     )
@@
       (effects (font (size 1.27 1.27)) hide)
     )
-    (property "LCSC" "" (at 87.63 31.75 0)
+    (property "LCSC" "C1511834" (at 87.63 31.75 0)
       (effects (font (size 1.27 1.27)) hide)
     )
@@
       (effects (font (size 1.27 1.27)) hide)
     )
-    (property "LCSC" "" (at 86.36 73.66 0)
+    (property "LCSC" "C3280240" (at 86.36 73.66 0)
       (effects (font (size 1.27 1.27)) hide)
     )
@@
       (effects (font (size 1.27 1.27)) hide)
     )
-    (property "LCSC" "" (at 71.12 68.58 0)
+    (property "LCSC" "C3280240" (at 71.12 68.58 0)
       (effects (font (size 1.27 1.27)) hide)
     )
@@
       (effects (font (size 1.27 1.27)) hide)
     )
-    (property "LCSC" "" (at 92.71 38.1 0)
+    (property "LCSC" "C1511834" (at 92.71 38.1 0)
       (effects (font (size 1.27 1.27)) hide)
     )
@@
       (effects (font (size 1.27 1.27)) hide)
     )
-    (property "LCSC" "" (at 45.72 114.3 0)
+    (property "LCSC" "C559075" (at 45.72 114.3 0)
       (effects (font (size 1.27 1.27)) hide)
     )
@@
       (effects (font (size 1.27 1.27)) hide)
     )
-    (property "LCSC" "" (at 50.8 151.13 0)
+    (property "LCSC" "C1589" (at 50.8 151.13 0)
       (effects (font (size 1.27 1.27)) hide)
     )
@@
       (effects (font (size 1.27 1.27)) hide)
     )
-    (property "LCSC" "" (at 45.72 105.41 0)
+    (property "LCSC" "C1511834" (at 45.72 105.41 0)
       (effects (font (size 1.27 1.27)) hide)
     )
@@
       (effects (font (size 1.27 1.27)) hide)
     )
-    (property "LCSC" "" (at 44.45 147.32 0)
+    (property "LCSC" "C3280240" (at 44.45 147.32 0)
       (effects (font (size 1.27 1.27)) hide)
     )
@@
       (effects (font (size 1.27 1.27)) hide)
     )
-    (property "LCSC" "" (at 29.21 142.24 0)
+    (property "LCSC" "C3280240" (at 29.21 142.24 0)
       (effects (font (size 1.27 1.27)) hide)
     )
@@
       (effects (font (size 1.27 1.27)) hide)
     )
-    (property "LCSC" "" (at 50.8 111.76 0)
+    (property "LCSC" "C1511834" (at 50.8 111.76 0)
       (effects (font (size 1.27 1.27)) hide)
     )
@@
       (effects (font (size 1.27 1.27)) hide)
     )
-    (property "LCSC" "" (at 87.63 114.3 0)
+    (property "LCSC" "C559075" (at 87.63 114.3 0)
       (effects (font (size 1.27 1.27)) hide)
     )
@@
       (effects (font (size 1.27 1.27)) hide)
     )
-    (property "LCSC" "" (at 92.71 151.13 0)
+    (property "LCSC" "C1589" (at 92.71 151.13 0)
       (effects (font (size 1.27 1.27)) hide)
     )
@@
       (effects (font (size 1.27 1.27)) hide)
     )
-    (property "LCSC" "" (at 87.63 105.41 0)
+    (property "LCSC" "C1511834" (at 87.63 105.41 0)
       (effects (font (size 1.27 1.27)) hide)
     )
@@
       (effects (font (size 1.27 1.27)) hide)
     )
-    (property "LCSC" "" (at 86.36 147.32 0)
+    (property "LCSC" "C3280240" (at 86.36 147.32 0)
       (effects (font (size 1.27 1.27)) hide)
     )
@@
       (effects (font (size 1.27 1.27)) hide)
     )
-    (property "LCSC" "" (at 71.12 142.24 0)
+    (property "LCSC" "C3280240" (at 71.12 142.24 0)
       (effects (font (size 1.27 1.27)) hide)
     )
@@
       (effects (font (size 1.27 1.27)) hide)
     )
-    (property "LCSC" "" (at 92.71 111.76 0)
+    (property "LCSC" "C1511834" (at 92.71 111.76 0)
       (effects (font (size 1.27 1.27)) hide)
     )
@@
       (effects (font (size 1.27 1.27)) hide)
     )
-    (property "LCSC" "" (at 45.72 132.08 0)
+    (property "LCSC" "C559075" (at 45.72 132.08 0)
       (effects (font (size 1.27 1.27)) hide)
     )
@@
       (effects (font (size 1.27 1.27)) hide)
     )
-    (property "LCSC" "" (at 87.63 132.08 0)
+    (property "LCSC" "C559075" (at 87.63 132.08 0)
       (effects (font (size 1.27 1.27)) hide)
     )
@@
       (effects (font (size 1.27 1.27)) hide)
     )
-    (property "LCSC" "" (at 209.55 105.41 0)
+    (property "LCSC" "C844773" (at 209.55 105.41 0)
       (effects (font (size 1.27 1.27)) hide)
     )
@@
       (effects (font (size 1.27 1.27)) hide)
     )
-    (property "LCSC" "" (at 208.28 31.75 0)
+    (property "LCSC" "C844773" (at 208.28 31.75 0)
       (effects (font (size 1.27 1.27)) hide)
     )
@@
       (effects (font (size 1.27 1.27)) hide)
     )
-    (property "LCSC" "" (at 213.36 72.39 0)
+    (property "LCSC" "C414226" (at 213.36 72.39 0)
       (effects (font (size 1.27 1.27)) hide)
     )
@@
       (effects (font (size 1.27 1.27)) hide)
     )
-    (property "LCSC" "" (at 212.09 36.83 0)
+    (property "LCSC" "C414226" (at 212.09 36.83 0)
       (effects (font (size 1.27 1.27)) hide)
     )
@@
       (effects (font (size 1.27 1.27)) hide)
     )
-    (property "LCSC" "" (at 213.36 110.49 0)
-      (effects (font (size 1.27 1.27)) hide)
-    )
+    (property "LCSC" "C2914421" (at 213.36 110.49 0)
+      (effects (font (size 1.27 1.27)) hide)
+    )

Commit message: edits
Parts:
- R71, R72, R86, R87: LCSC (none) -> C4244464
- R75, R76, R95, R96: LCSC (none) -> C105580
Changed lines of the file:
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@@
       (effects (font (size 1.27 1.27)) hide)
     )
-    (property "LCSC" "" (at 39.37 53.34 0)
+    (property "LCSC" "C4244464" (at 39.37 53.34 0)
       (effects (font (size 1.27 1.27)) hide)
     )
@@
       (effects (font (size 1.27 1.27)) hide)
     )
-    (property "LCSC" "" (at 50.8 67.31 0)
+    (property "LCSC" "C105580" (at 50.8 67.31 0)
       (effects (font (size 1.27 1.27)) hide)
     )
@@
       (effects (font (size 1.27 1.27)) hide)
     )
-    (property "LCSC" "" (at 81.28 53.34 0)
+    (property "LCSC" "C4244464" (at 81.28 53.34 0)
       (effects (font (size 1.27 1.27)) hide)
     )
@@
       (effects (font (size 1.27 1.27)) hide)
     )
-    (property "LCSC" "" (at 92.71 67.31 0)
+    (property "LCSC" "C105580" (at 92.71 67.31 0)
       (effects (font (size 1.27 1.27)) hide)
     )
@@
       (effects (font (size 1.27 1.27)) hide)
     )
-    (property "LCSC" "" (at 39.37 127 0)
+    (property "LCSC" "C4244464" (at 39.37 127 0)
       (effects (font (size 1.27 1.27)) hide)
     )
@@
       (effects (font (size 1.27 1.27)) hide)
     )
-    (property "LCSC" "" (at 50.8 140.97 0)
+    (property "LCSC" "C105580" (at 50.8 140.97 0)
       (effects (font (size 1.27 1.27)) hide)
     )
@@
       (effects (font (size 1.27 1.27)) hide)
     )
-    (property "LCSC" "" (at 81.28 127 0)
+    (property "LCSC" "C4244464" (at 81.28 127 0)
       (effects (font (size 1.27 1.27)) hide)
     )
@@
       (effects (font (size 1.27 1.27)) hide)
     )
-    (property "LCSC" "" (at 92.71 140.97 0)
-      (effects (font (size 1.27 1.27)) hide)
-    )
+    (property "LCSC" "C105580" (at 92.71 140.97 0)
+      (effects (font (size 1.27 1.27)) hide)
+    )

Commit message: Improved Py-Cubed BOM
Parts:
- R101, R104, R107, R108, R109, R48, R53, R97, R98, R99: LCSC (none) -> C2654002
- R63, R64, R69, R70, R77, R78: LCSC (none) -> C844746
- R68: LCSC (none) -> C844773
- R73, R74, R93, R94: LCSC (none) -> C5369222
- R75, R76, R95, R96: LCSC C105580 -> C1854765
Changed lines of the file:
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@@
       (effects (font (size 1.27 1.27)) hide)
     )
-    (property "LCSC" "" (at 38.1 64.77 0)
+    (property "LCSC" "C5369222" (at 38.1 64.77 0)
       (effects (font (size 1.27 1.27)) hide)
     )
@@
       (effects (font (size 1.27 1.27)) hide)
     )
-    (property "LCSC" "C105580" (at 50.8 67.31 0)
+    (property "LCSC" "C1854765" (at 50.8 67.31 0)
       (effects (font (size 1.27 1.27)) hide)
     )
@@
       (effects (font (size 1.27 1.27)) hide)
     )
-    (property "LCSC" "C105580" (at 92.71 67.31 0)
+    (property "LCSC" "C1854765" (at 92.71 67.31 0)
       (effects (font (size 1.27 1.27)) hide)
     )
@@
       (effects (font (size 1.27 1.27)) hide)
     )
-    (property "LCSC" "" (at 80.01 64.77 0)
+    (property "LCSC" "C5369222" (at 80.01 64.77 0)
       (effects (font (size 1.27 1.27)) hide)
     )
@@
       (effects (font (size 1.27 1.27)) hide)
     )
-    (property "LCSC" "C105580" (at 50.8 140.97 0)
+    (property "LCSC" "C1854765" (at 50.8 140.97 0)
       (effects (font (size 1.27 1.27)) hide)
     )
@@
       (effects (font (size 1.27 1.27)) hide)
     )
-    (property "LCSC" "" (at 38.1 138.43 0)
+    (property "LCSC" "C5369222" (at 38.1 138.43 0)
       (effects (font (size 1.27 1.27)) hide)
     )
@@
       (effects (font (size 1.27 1.27)) hide)
     )
-    (property "LCSC" "C105580" (at 92.71 140.97 0)
+    (property "LCSC" "C1854765" (at 92.71 140.97 0)
       (effects (font (size 1.27 1.27)) hide)
     )
@@
       (effects (font (size 1.27 1.27)) hide)
     )
-    (property "LCSC" "" (at 80.01 138.43 0)
+    (property "LCSC" "C5369222" (at 80.01 138.43 0)
       (effects (font (size 1.27 1.27)) hide)
     )
@@
       (effects (font (size 1.27 1.27)) hide)
     )
-    (property "LCSC" "" (at 209.55 67.31 0)
+    (property "LCSC" "C844773" (at 209.55 67.31 0)
       (effects (font (size 1.27 1.27)) hide)
     )
@@
       (effects (font (size 1.27 1.27)) hide)
     )
-    (property "LCSC" "" (at 237.49 30.48 0)
+    (property "LCSC" "C844746" (at 237.49 30.48 0)
       (effects (font (size 1.27 1.27)) hide)
     )
@@
       (effects (font (size 1.27 1.27)) hide)
     )
-    (property "LCSC" "" (at 237.49 66.04 0)
+    (property "LCSC" "C844746" (at 237.49 66.04 0)
       (effects (font (size 1.27 1.27)) hide)
     )
@@
       (effects (font (size 1.27 1.27)) hide)
     )
-    (property "LCSC" "" (at 237.49 39.37 0)
+    (property "LCSC" "C844746" (at 237.49 39.37 0)
       (effects (font (size 1.27 1.27)) hide)
     )
@@
       (effects (font (size 1.27 1.27)) hide)
     )
-    (property "LCSC" "" (at 237.49 113.03 0)
+    (property "LCSC" "C844746" (at 237.49 113.03 0)
       (effects (font (size 1.27 1.27)) hide)
     )
@@
       (effects (font (size 1.27 1.27)) hide)
     )
-    (property "LCSC" "" (at 237.49 104.14 0)
+    (property "LCSC" "C844746" (at 237.49 104.14 0)
       (effects (font (size 1.27 1.27)) hide)
     )
@@
       (effects (font (size 1.27 1.27)) hide)
     )
-    (property "LCSC" "" (at 67.31 193.04 0)
+    (property "LCSC" "C2654002" (at 67.31 193.04 0)
       (effects (font (size 1.27 1.27)) hide)
     )
@@
       (effects (font (size 1.27 1.27)) hide)
     )
-    (property "LCSC" "" (at 67.31 179.07 0)
+    (property "LCSC" "C2654002" (at 67.31 179.07 0)
       (effects (font (size 1.27 1.27)) hide)
     )
@@
       (effects (font (size 1.27 1.27)) hide)
     )
-    (property "LCSC" "" (at 67.31 182.88 0)
+    (property "LCSC" "C2654002" (at 67.31 182.88 0)
       (effects (font (size 1.27 1.27)) hide)
     )
@@
       (effects (font (size 1.27 1.27)) hide)
     )
-    (property "LCSC" "" (at 102.87 185.42 0)
+    (property "LCSC" "C2654002" (at 102.87 185.42 0)
       (effects (font (size 1.27 1.27)) hide)
     )
@@
       (effects (font (size 1.27 1.27)) hide)
     )
-    (property "LCSC" "" (at 102.87 190.5 0)
+    (property "LCSC" "C2654002" (at 102.87 190.5 0)
       (effects (font (size 1.27 1.27)) hide)
     )
@@
       (effects (font (size 1.27 1.27)) hide)
     )
-    (property "LCSC" "" (at 67.31 189.23 0)
+    (property "LCSC" "C2654002" (at 67.31 189.23 0)
       (effects (font (size 1.27 1.27)) hide)
     )
@@
       (effects (font (size 1.27 1.27)) hide)
     )
-    (property "LCSC" "" (at 102.87 180.34 0)
+    (property "LCSC" "C2654002" (at 102.87 180.34 0)
       (effects (font (size 1.27 1.27)) hide)
     )
@@
       (effects (font (size 1.27 1.27)) hide)
     )
-    (property "LCSC" "" (at 204.47 74.93 0)
+    (property "LCSC" "C2654002" (at 204.47 74.93 0)
       (effects (font (size 1.27 1.27)) hide)
     )
@@
       (effects (font (size 1.27 1.27)) hide)
     )
-    (property "LCSC" "" (at 237.49 74.93 0)
+    (property "LCSC" "C844746" (at 237.49 74.93 0)
       (effects (font (size 1.27 1.27)) hide)
     )
@@
       (effects (font (size 1.27 1.27)) hide)
     )
-    (property "LCSC" "" (at 204.47 113.03 0)
+    (property "LCSC" "C2654002" (at 204.47 113.03 0)
       (effects (font (size 1.27 1.27)) hide)
     )
@@
       (effects (font (size 1.27 1.27)) hide)
     )
-    (property "LCSC" "" (at 203.2 39.37 0)
-      (effects (font (size 1.27 1.27)) hide)
-    )
+    (property "LCSC" "C2654002" (at 203.2 39.37 0)
+      (effects (font (size 1.27 1.27)) hide)
+    )
