File: mainboard-v05/Connectors.kicad_sch (KiCad schematic)
At the start: 18 parts, among them J1 503182-1852, J11 10118194-0001LF, J13 USB_C_Receptacle_USB2.0, J16 1985807, J17 1985807, J18 1985807, J2 Conn_01x05, J3 1985807, J4 1985807, U8 MR25H40MDF

Commit message: Added more fields to BOM.
Parts:
- C24, C30: LCSC (none) -> C1591
- C29: LCSC (none) -> C1705
- C31: LCSC (none) -> C59461
Changed lines of the file:
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@@
       (effects (font (size 1.27 1.27)) hide)
     )
-    (property "LCSC" "" (at 80.01 116.84 0)
+    (property "LCSC" "C1591" (at 80.01 116.84 0)
       (effects (font (size 1.27 1.27)) hide)
     )
@@
       (effects (font (size 1.27 1.27)) hide)
     )
-    (property "LCSC" "" (at 224.79 57.15 0)
+    (property "LCSC" "C1591" (at 224.79 57.15 0)
       (effects (font (size 1.27 1.27)) hide)
     )
@@
       (effects (font (size 1.27 1.27)) hide)
     )
-    (property "LCSC" "" (at 234.95 57.15 0)
+    (property "LCSC" "C59461" (at 234.95 57.15 0)
       (effects (font (size 1.27 1.27)) hide)
     )
@@
       (effects (font (size 1.27 1.27)) hide)
     )
-    (property "LCSC" "" (at 179.07 73.66 0)
-      (effects (font (size 1.27 1.27)) hide)
-    )
+    (property "LCSC" "C1705" (at 179.07 73.66 0)
+      (effects (font (size 1.27 1.27)) hide)
+    )

Commit message: edits
Parts:
- R39, R40: renamed from R?; LCSC (none) -> C185333
- U8: LCSC (none) -> NotAvailable
- gave numbers to parts that had none: 2
Changed lines of the file:
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@@
           (reference "#GND022") (unit 1)
         )
-        (path "/e3ac22ea-6806-4807-a025-571315789c25"
-          (reference "#GND?") (unit 1)
-        )
       )
     )
@@
         (path "/e3ac22ea-6806-4807-a025-571315789c25/00000000-0000-0000-0000-00005cec60eb"
           (reference "J3") (unit 1)
-        )
-        (path "/e3ac22ea-6806-4807-a025-571315789c25"
-          (reference "JP?") (unit 1)
         )
       )
@@
           (reference "J1") (unit 1)
         )
-        (path "/e3ac22ea-6806-4807-a025-571315789c25"
-          (reference "J?") (unit 1)
-        )
       )
     )
@@
       (effects (font (size 1.27 1.27)) hide)
     )
-    (property "LCSC" "" (at 41.91 119.38 0)
+    (property "LCSC" "NotAvailable" (at 41.91 119.38 0)
       (effects (font (size 1.27 1.27)) hide)
     )
@@
           (reference "U8") (unit 1)
         )
-        (path "/e3ac22ea-6806-4807-a025-571315789c25"
-          (reference "U?") (unit 1)
-        )
       )
     )
@@
         (path "/e3ac22ea-6806-4807-a025-571315789c25/00000000-0000-0000-0000-00005cec60eb"
           (reference "J4") (unit 1)
-        )
-        (path "/e3ac22ea-6806-4807-a025-571315789c25"
-          (reference "JP?") (unit 1)
         )
       )
@@
           (reference "C30") (unit 1)
         )
-        (path "/e3ac22ea-6806-4807-a025-571315789c25"
-          (reference "C?") (unit 1)
-        )
       )
     )
@@
           (reference "#GND065") (unit 1)
         )
-        (path "/e3ac22ea-6806-4807-a025-571315789c25"
-          (reference "#GND?") (unit 1)
-        )
       )
     )
@@
         (path "/e3ac22ea-6806-4807-a025-571315789c25/00000000-0000-0000-0000-00005cec60eb"
           (reference "#GND023") (unit 1)
-        )
-        (path "/e3ac22ea-6806-4807-a025-571315789c25"
-          (reference "#GND?") (unit 1)
         )
       )
@@
         (path "/e3ac22ea-6806-4807-a025-571315789c25/00000000-0000-0000-0000-00005cec60eb"
           (reference "#SUPPLY0102") (unit 1)
-        )
-        (path "/e3ac22ea-6806-4807-a025-571315789c25"
-          (reference "#SUPPLY?") (unit 1)
         )
       )
@@
     (instances
       (project "mainboard"
-        (path "/e3ac22ea-6806-4807-a025-571315789c25"
-          (reference "J13") (unit 1)
-        )
         (path "/e3ac22ea-6806-4807-a025-571315789c25/00000000-0000-0000-0000-00005cec60eb"
           (reference "J13") (unit 1)
@@
           (reference "C24") (unit 1)
         )
-        (path "/e3ac22ea-6806-4807-a025-571315789c25/00000000-0000-0000-0000-00005cec5dde"
-          (reference "C?") (unit 1)
-        )
       )
     )
@@
           (reference "C31") (unit 1)
         )
-        (path "/e3ac22ea-6806-4807-a025-571315789c25/00000000-0000-0000-0000-00005cec5dde"
-          (reference "C?") (unit 1)
-        )
       )
     )
@@
   (symbol (lib_id "Device:R_US") (at 64.77 34.29 0) (mirror x) (unit 1)
     (in_bom yes) (on_board yes) (dnp no)
-    (property "Reference" "R?" (at 62.23 31.75 0)
+    (property "Reference" "R51" (at 62.23 31.75 0)
       (effects (font (size 1.27 1.27)))
     )
@@
     (instances
       (project "mainboard"
-        (path "/e3ac22ea-6806-4807-a025-571315789c25/00000000-0000-0000-0000-00005cec5dde"
-          (reference "R?") (unit 1)
-        )
-        (path "/e3ac22ea-6806-4807-a025-571315789c25/00000000-0000-0000-0000-00005cec5a72"
-          (reference "R?") (unit 1)
-        )
         (path "/e3ac22ea-6806-4807-a025-571315789c25/00000000-0000-0000-0000-00005cec60eb"
           (reference "R51") (unit 1)
@@
           (reference "J17") (unit 1)
         )
-        (path "/e3ac22ea-6806-4807-a025-571315789c25"
-          (reference "JP?") (unit 1)
-        )
       )
     )
@@
   (symbol (lib_id "Device:R_US") (at 35.56 115.57 0) (mirror x) (unit 1)
     (in_bom yes) (on_board yes) (dnp no)
-    (property "Reference" "R?" (at 33.02 113.03 0)
+    (property "Reference" "R50" (at 33.02 113.03 0)
       (effects (font (size 1.27 1.27)))
     )
@@
     (instances
       (project "mainboard"
-        (path "/e3ac22ea-6806-4807-a025-571315789c25/00000000-0000-0000-0000-00005cec5dde"
-          (reference "R?") (unit 1)
-        )
-        (path "/e3ac22ea-6806-4807-a025-571315789c25/00000000-0000-0000-0000-00005cec5a72"
-          (reference "R?") (unit 1)
-        )
         (path "/e3ac22ea-6806-4807-a025-571315789c25/00000000-0000-0000-0000-00005cec60eb"
           (reference "R50") (unit 1)
@@
           (reference "#SUPPLY0116") (unit 1)
         )
-        (path "/e3ac22ea-6806-4807-a025-571315789c25"
-          (reference "#SUPPLY?") (unit 1)
-        )
       )
     )
@@
   (symbol (lib_id "Device:R_US") (at 157.48 59.69 0) (mirror x) (unit 1)
     (in_bom yes) (on_board yes) (dnp no)
-    (property "Reference" "R?" (at 154.94 57.15 0)
+    (property "Reference" "R40" (at 154.94 57.15 0)
       (effects (font (size 1.27 1.27)))
     )
@@
       (effects (font (size 1.27 1.27)) hide)
     )
-    (property "LCSC" "" (at 157.48 59.69 0)
-      (effects (font (size 1.27 1.27)) hide)
-    )
-    (pin "1")
-    (pin "2")
-    (instances
-      (project "mainboard"
-        (path "/e3ac22ea-6806-4807-a025-571315789c25/00000000-0000-0000-0000-00005cec5dde"
-          (reference "R?") (unit 1)
-        )
-        (path "/e3ac22ea-6806-4807-a025-571315789c25/00000000-0000-0000-0000-00005cec5a72"
-          (reference "R?") (unit 1)
-        )
+    (property "LCSC" "C185333" (at 157.48 59.69 0)
+      (effects (font (size 1.27 1.27)) hide)
+    )
+    (pin "1")
+    (pin "2")
+    (instances
+      (project "mainboard"
         (path "/e3ac22ea-6806-4807-a025-571315789c25/00000000-0000-0000-0000-00005cec60eb"
           (reference "R40") (unit 1)
@@
   (symbol (lib_id "Device:R_US") (at 154.94 62.23 0) (mirror x) (unit 1)
     (in_bom yes) (on_board yes) (dnp no)
-    (property "Reference" "R?" (at 152.4 59.69 0)
+    (property "Reference" "R39" (at 152.4 59.69 0)
       (effects (font (size 1.27 1.27)))
     )
@@
       (effects (font (size 1.27 1.27)) hide)
     )
-    (property "LCSC" "" (at 154.94 62.23 0)
-      (effects (font (size 1.27 1.27)) hide)
-    )
-    (pin "1")
-    (pin "2")
-    (instances
-      (project "mainboard"
-        (path "/e3ac22ea-6806-4807-a025-571315789c25/00000000-0000-0000-0000-00005cec5dde"
-          (reference "R?") (unit 1)
-        )
-        (path "/e3ac22ea-6806-4807-a025-571315789c25/00000000-0000-0000-0000-00005cec5a72"
-          (reference "R?") (unit 1)
-        )
+    (property "LCSC" "C185333" (at 154.94 62.23 0)
+      (effects (font (size 1.27 1.27)) hide)
+    )
+    (pin "1")
+    (pin "2")
+    (instances
+      (project "mainboard"
         (path "/e3ac22ea-6806-4807-a025-571315789c25/00000000-0000-0000-0000-00005cec60eb"
           (reference "R39") (unit 1)
@@
         (path "/e3ac22ea-6806-4807-a025-571315789c25/00000000-0000-0000-0000-00005cec60eb"
           (reference "#PWR0107") (unit 1)
-        )
-        (path "/e3ac22ea-6806-4807-a025-571315789c25/00000000-0000-0000-0000-00005cec5dde"
-          (reference "#PWR?") (unit 1)
         )
       )
@@
           (reference "#PWR0108") (unit 1)
         )
-        (path "/e3ac22ea-6806-4807-a025-571315789c25/00000000-0000-0000-0000-00005cec5dde"
-          (reference "#PWR?") (unit 1)
-        )
       )
     )
@@
           (reference "C29") (unit 1)
         )
-        (path "/e3ac22ea-6806-4807-a025-571315789c25/00000000-0000-0000-0000-00005cec5dde"
-          (reference "C?") (unit 1)
-        )
       )
     )
@@
           (reference "#PWR0101") (unit 1)
         )
-        (path "/e3ac22ea-6806-4807-a025-571315789c25/00000000-0000-0000-0000-00005cec5dde"
-          (reference "#PWR?") (unit 1)
-        )
       )
     )
@@
           (reference "#PWR0109") (unit 1)
         )
-        (path "/e3ac22ea-6806-4807-a025-571315789c25/00000000-0000-0000-0000-00005cec5dde"
-          (reference "#PWR?") (unit 1)
-        )
       )
     )
@@
         (path "/e3ac22ea-6806-4807-a025-571315789c25/00000000-0000-0000-0000-00005cec60eb"
           (reference "#GND025") (unit 1)
-        )
-        (path "/e3ac22ea-6806-4807-a025-571315789c25"
-          (reference "#GND?") (unit 1)
         )
       )
@@
           (reference "J16") (unit 1)
         )
-        (path "/e3ac22ea-6806-4807-a025-571315789c25"
-          (reference "JP?") (unit 1)
-        )
       )
     )
@@
           (reference "#SUPPLY08") (unit 1)
         )
-        (path "/e3ac22ea-6806-4807-a025-571315789c25"
-          (reference "#SUPPLY?") (unit 1)
-        )
       )
     )
@@
           (reference "#GND029") (unit 1)
         )
-        (path "/e3ac22ea-6806-4807-a025-571315789c25"
-          (reference "#GND?") (unit 1)
-        )
       )
     )
@@
           (reference "#GND026") (unit 1)
         )
-        (path "/e3ac22ea-6806-4807-a025-571315789c25"
-          (reference "#GND?") (unit 1)
-        )
       )
     )
@@
           (reference "#GND024") (unit 1)
         )
-        (path "/e3ac22ea-6806-4807-a025-571315789c25"
-          (reference "#GND?") (unit 1)
-        )
       )
     )
@@
           (reference "#SUPPLY07") (unit 1)
         )
-        (path "/e3ac22ea-6806-4807-a025-571315789c25"
-          (reference "#SUPPLY?") (unit 1)
-        )
       )
     )
@@
           (reference "J18") (unit 1)
         )
-        (path "/e3ac22ea-6806-4807-a025-571315789c25"
-          (reference "JP?") (unit 1)
-        )
-      )
+      )

Commit message: Improved Py-Cubed BOM
Parts:
- J1, J13, J16, J17, J18, J3, J4: LCSC (none) -> NotAvailable
- J2: LCSC (none) -> C2883762
- R39, R40: LCSC C185333 -> C105580
- R50, R51: LCSC (none) -> C1511834
Changed lines of the file:
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@@
       (effects (font (size 1.27 1.27)) hide)
     )
-    (property "LCSC" "" (at 201.93 52.07 0)
+    (property "LCSC" "NotAvailable" (at 201.93 52.07 0)
       (effects (font (size 1.27 1.27)) hide)
     )
@@
       (effects (font (size 1.27 1.27)) hide)
     )
-    (property "LCSC" "" (at 53.34 50.8 0)
+    (property "LCSC" "NotAvailable" (at 53.34 50.8 0)
       (effects (font (size 1.27 1.27)) hide)
     )
@@
       (effects (font (size 1.27 1.27)) hide)
     )
-    (property "LCSC" "" (at 201.93 67.31 0)
+    (property "LCSC" "NotAvailable" (at 201.93 67.31 0)
       (effects (font (size 1.27 1.27)) hide)
     )
@@
       (effects (font (size 1.27 1.27)) hide)
     )
-    (property "LCSC" "" (at 69.85 168.91 0)
+    (property "LCSC" "C2883762" (at 69.85 168.91 0)
       (effects (font (size 1.27 1.27)) hide)
     )
@@
       (effects (font (size 1.27 1.27)) hide)
     )
-    (property "LCSC" "" (at 123.19 66.04 0)
+    (property "LCSC" "NotAvailable" (at 123.19 66.04 0)
       (effects (font (size 1.27 1.27)) hide)
     )
@@
       (effects (font (size 1.27 1.27)) hide)
     )
-    (property "LCSC" "" (at 64.77 34.29 0)
+    (property "LCSC" "C1511834" (at 64.77 34.29 0)
       (effects (font (size 1.27 1.27)) hide)
     )
@@
       (effects (font (size 1.27 1.27)) hide)
     )
-    (property "LCSC" "" (at 254 83.82 0)
+    (property "LCSC" "NotAvailable" (at 254 83.82 0)
       (effects (font (size 1.27 1.27)) hide)
     )
@@
       (effects (font (size 1.27 1.27)) hide)
     )
-    (property "LCSC" "" (at 35.56 115.57 0)
+    (property "LCSC" "C1511834" (at 35.56 115.57 0)
       (effects (font (size 1.27 1.27)) hide)
     )
@@
       (effects (font (size 1.27 1.27)) hide)
     )
-    (property "LCSC" "C185333" (at 157.48 59.69 0)
+    (property "LCSC" "C105580" (at 157.48 59.69 0)
       (effects (font (size 1.27 1.27)) hide)
     )
@@
       (effects (font (size 1.27 1.27)) hide)
     )
-    (property "LCSC" "C185333" (at 154.94 62.23 0)
+    (property "LCSC" "C105580" (at 154.94 62.23 0)
       (effects (font (size 1.27 1.27)) hide)
     )
@@
       (effects (font (size 1.27 1.27)) hide)
     )
-    (property "LCSC" "" (at 242.57 83.82 0)
+    (property "LCSC" "NotAvailable" (at 242.57 83.82 0)
       (effects (font (size 1.27 1.27)) hide)
     )
@@
       (effects (font (size 1.27 1.27)) hide)
     )
-    (property "LCSC" "" (at 207.01 93.98 0)
-      (effects (font (size 1.27 1.27)) hide)
-    )
+    (property "LCSC" "NotAvailable" (at 207.01 93.98 0)
+      (effects (font (size 1.27 1.27)) hide)
+    )
