File: mainboard-v05/Power.kicad_sch (KiCad schematic)
At the start: 70 parts, among them J14 Conn_01x06, Q1 IRLML2803, Q2 MBT2222ADW1T1, Q22 NDS8434, Q3 MBT2222ADW1T1, U17 BQ25883RGER, U21 TPS7A4501DCQT, U4 ADM1176-1ARMZ-R7, U5 TPS54226PWPRPWP14_2P31X2P46-L, U6 LTC4121, U7 KF50BD-TR

Commit message: Added more fields to BOM.
Parts:
- C17, C18, C28, C37, C38: LCSC (none) -> C59461
- C19, C20: LCSC (none) -> C49066
- C21, C45: LCSC (none) -> C1591
- C22, C35, C39, C43, C6: LCSC (none) -> C1691
- C23: LCSC (none) -> C23630
- C25: LCSC (none) -> C21122
- C26, C32: LCSC (none) -> C1613
- C27, C33: LCSC (none) -> C1592
- C34: LCSC (none) -> C1705
- C36: LCSC (none) -> C1622
- D2: LCSC (none) -> C5380706
- Q1: LCSC (none) -> C2590
- Q2, Q3: LCSC (none) -> C559075
- R21, R31, R46, R52, R55: LCSC (none) -> C1511834
- R8: LCSC (none) -> C4240903
Changed lines of the file:
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@@
       (effects (font (size 1.27 1.27)) hide)
     )
-    (property "LCSC" "" (at 57.15 173.99 0)
+    (property "LCSC" "C1591" (at 57.15 173.99 0)
       (effects (font (size 1.27 1.27)) hide)
     )
@@
       (effects (font (size 1.27 1.27) bold))
     )
-    (property "LCSC" "" (at 31.75 46.99 0)
+    (property "LCSC" "C5380706" (at 31.75 46.99 0)
       (effects (font (size 1.27 1.27)) hide)
     )
@@
       (effects (font (size 1.27 1.27)) hide)
     )
-    (property "LCSC" "" (at 46.99 57.15 0)
+    (property "LCSC" "C1691" (at 46.99 57.15 0)
       (effects (font (size 1.27 1.27)) hide)
     )
@@
       (effects (font (size 1.27 1.27)) hide)
     )
-    (property "LCSC" "" (at 119.38 100.33 0)
+    (property "LCSC" "C4240903" (at 119.38 100.33 0)
       (effects (font (size 1.27 1.27)) hide)
     )
@@
       (effects (font (size 1.27 1.27)) hide)
     )
-    (property "LCSC" "" (at 231.14 55.88 0)
+    (property "LCSC" "C2590" (at 231.14 55.88 0)
       (effects (font (size 1.27 1.27)) hide)
     )
@@
       (effects (font (size 1.27 1.27)) hide)
     )
-    (property "LCSC" "" (at 148.59 189.23 0)
+    (property "LCSC" "C1592" (at 148.59 189.23 0)
       (effects (font (size 1.27 1.27)) hide)
     )
@@
       (effects (font (size 1.27 1.27)) hide)
     )
-    (property "LCSC" "" (at 29.21 163.83 0)
+    (property "LCSC" "C59461" (at 29.21 163.83 0)
       (effects (font (size 1.27 1.27)) hide)
     )
@@
       (effects (font (size 1.27 1.27)) hide)
     )
-    (property "LCSC" "" (at 138.43 67.31 0)
+    (property "LCSC" "C59461" (at 138.43 67.31 0)
       (effects (font (size 1.27 1.27)) hide)
     )
@@
       (effects (font (size 1.27 1.27)) hide)
     )
-    (property "LCSC" "" (at 243.84 138.43 0)
+    (property "LCSC" "C1622" (at 243.84 138.43 0)
       (effects (font (size 1.27 1.27)) hide)
     )
@@
       (effects (font (size 1.27 1.27)) hide)
     )
-    (property "LCSC" "" (at 250.19 119.38 0)
+    (property "LCSC" "C59461" (at 250.19 119.38 0)
       (effects (font (size 1.27 1.27)) hide)
     )
@@
       (effects (font (size 1.27 1.27)) hide)
     )
-    (property "LCSC" "" (at 254 130.81 0)
+    (property "LCSC" "C1691" (at 254 130.81 0)
       (effects (font (size 1.27 1.27)) hide)
     )
@@
       (effects (font (size 1.27 1.27)) hide)
     )
-    (property "LCSC" "" (at 232.41 146.05 0)
+    (property "LCSC" "C1511834" (at 232.41 146.05 0)
       (effects (font (size 1.27 1.27)) hide)
     )
@@
       (effects (font (size 1.27 1.27)) hide)
     )
-    (property "LCSC" "" (at 212.09 146.05 0)
+    (property "LCSC" "C1705" (at 212.09 146.05 0)
       (effects (font (size 1.27 1.27)) hide)
     )
@@
       (effects (font (size 1.27 1.27)) hide)
     )
-    (property "LCSC" "" (at 205.74 86.36 0)
+    (property "LCSC" "C1592" (at 205.74 86.36 0)
       (effects (font (size 1.27 1.27)) hide)
     )
@@
       (effects (font (size 1.27 1.27)) hide)
     )
-    (property "LCSC" "" (at 237.49 86.36 0)
+    (property "LCSC" "C1691" (at 237.49 86.36 0)
       (effects (font (size 1.27 1.27)) hide)
     )
@@
       (effects (font (size 1.27 1.27)) hide)
     )
-    (property "LCSC" "" (at 254 119.38 0)
+    (property "LCSC" "C59461" (at 254 119.38 0)
       (effects (font (size 1.27 1.27)) hide)
     )
@@
       (effects (font (size 1.27 1.27)) hide)
     )
-    (property "LCSC" "" (at 172.72 95.25 0)
+    (property "LCSC" "C1613" (at 172.72 95.25 0)
       (effects (font (size 1.27 1.27)) hide)
     )
@@
       (effects (font (size 1.27 1.27)) hide)
     )
-    (property "LCSC" "" (at 208.28 142.24 0)
+    (property "LCSC" "C1511834" (at 208.28 142.24 0)
       (effects (font (size 1.27 1.27)) hide)
     )
@@
       (effects (font (size 1.27 1.27)) hide)
     )
-    (property "LCSC" "" (at 158.75 147.32 0)
+    (property "LCSC" "C559075" (at 158.75 147.32 0)
       (effects (font (size 1.27 1.27)) hide)
     )
@@
       (effects (font (size 1.27 1.27)) hide)
     )
-    (property "LCSC" "" (at 144.78 142.24 0)
+    (property "LCSC" "C559075" (at 144.78 142.24 0)
       (effects (font (size 1.27 1.27)) hide)
     )
@@
       (effects (font (size 1.27 1.27)) hide)
     )
-    (property "LCSC" "" (at 133.35 153.67 0)
+    (property "LCSC" "C559075" (at 133.35 153.67 0)
       (effects (font (size 1.27 1.27)) hide)
     )
@@
       (effects (font (size 1.27 1.27)) hide)
     )
-    (property "LCSC" "" (at 171.45 147.32 0)
+    (property "LCSC" "C559075" (at 171.45 147.32 0)
       (effects (font (size 1.27 1.27)) hide)
     )
@@
       (effects (font (size 1.27 1.27)) hide)
     )
-    (property "LCSC" "" (at 176.53 151.13 0)
+    (property "LCSC" "C1511834" (at 176.53 151.13 0)
       (effects (font (size 1.27 1.27)) hide)
     )
@@
       (effects (font (size 1.27 1.27)) hide)
     )
-    (property "LCSC" "" (at 36.83 181.61 0)
+    (property "LCSC" "C49066" (at 36.83 181.61 0)
       (effects (font (size 1.27 1.27)) hide)
     )
@@
       (effects (font (size 1.27 1.27)) hide)
     )
-    (property "LCSC" "" (at 153.67 142.24 0)
+    (property "LCSC" "C1691" (at 153.67 142.24 0)
       (effects (font (size 1.27 1.27)) hide)
     )
@@
       (effects (font (size 1.27 1.27)) hide)
     )
-    (property "LCSC" "" (at 44.45 113.03 0)
+    (property "LCSC" "C1691" (at 44.45 113.03 0)
       (effects (font (size 1.27 1.27)) hide)
     )
@@
       (effects (font (size 1.27 1.27)) hide)
     )
-    (property "LCSC" "" (at 49.53 115.57 0)
+    (property "LCSC" "C1511834" (at 49.53 115.57 0)
       (effects (font (size 1.27 1.27)) hide)
     )
@@
       (effects (font (size 1.27 1.27)) hide)
     )
-    (property "LCSC" "" (at 95.25 135.89 0)
+    (property "LCSC" "C1591" (at 95.25 135.89 0)
       (effects (font (size 1.27 1.27)) hide)
     )
@@
       (effects (font (size 1.27 1.27)) hide)
     )
-    (property "LCSC" "" (at 140.97 173.99 0)
+    (property "LCSC" "C1613" (at 140.97 173.99 0)
       (effects (font (size 1.27 1.27)) hide)
     )
@@
       (effects (font (size 1.27 1.27)) hide)
     )
-    (property "LCSC" "" (at 215.9 55.88 0)
+    (property "LCSC" "C1511834" (at 215.9 55.88 0)
       (effects (font (size 1.27 1.27)) hide)
     )
@@
       (effects (font (size 1.27 1.27)) hide)
     )
-    (property "LCSC" "" (at 77.47 49.53 0)
+    (property "LCSC" "C21122" (at 77.47 49.53 0)
       (effects (font (size 1.27 1.27)) hide)
     )
@@
       (effects (font (size 1.27 1.27)) hide)
     )
-    (property "LCSC" "" (at 36.83 163.83 0)
+    (property "LCSC" "C59461" (at 36.83 163.83 0)
       (effects (font (size 1.27 1.27)) hide)
     )
@@
       (effects (font (size 1.27 1.27)) hide)
     )
-    (property "LCSC" "" (at 46.99 181.61 0)
+    (property "LCSC" "C49066" (at 46.99 181.61 0)
       (effects (font (size 1.27 1.27)) hide)
     )
@@
       (effects (font (size 1.27 1.27)) hide)
     )
-    (property "LCSC" "" (at 77.47 36.83 0)
+    (property "LCSC" "C23630" (at 77.47 36.83 0)
       (effects (font (size 1.27 1.27)) hide)
     )

Commit message: edits
Parts:
- R110: LCSC (none) -> C2076573
- R47: LCSC (none) -> C105580
- U17, U21, U4, U5, U7: LCSC (none) -> NotAvailable
- U6: LCSC (none) -> C687336

Commit message: Improved Py-Cubed BOM
Parts:
- D5, L2, L3, L4, Q22: LCSC (none) -> NotAvailable
- J14: LCSC (none) -> C2883763
- R10: LCSC (none) -> C2654002
- R11: LCSC (none) -> C246008
- R12: LCSC (none) -> C2992526
- R13, R29: LCSC (none) -> C844180
- R14: LCSC (none) -> C844759
- R15, R17, R18, R30, R49: LCSC (none) -> C5369222
- R16: LCSC (none) -> C2091473
- R19: LCSC (none) -> C2085910
- R20: LCSC (none) -> C2075334
- R22: LCSC (none) -> C844773
- R23, R59: LCSC (none) -> C844782
- R26: LCSC (none) -> C844746
- R34: LCSC (none) -> C849180
- R35: LCSC (none) -> C844775
- R36: LCSC (none) -> C185333
- R47: LCSC C105580 -> C1854765
Changed lines of the file:
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@@
       (effects (font (size 1.27 1.27)) hide)
     )
-    (property "LCSC" "" (at 138.43 186.69 0)
+    (property "LCSC" "C844759" (at 138.43 186.69 0)
       (effects (font (size 1.27 1.27)) hide)
     )
@@
       (effects (font (size 1.27 1.27)) hide)
     )
-    (property "LCSC" "" (at 138.43 34.29 0)
+    (property "LCSC" "C5369222" (at 138.43 34.29 0)
       (effects (font (size 1.27 1.27)) hide)
     )
@@
       (effects (font (size 1.27 1.27)) hide)
     )
-    (property "LCSC" "" (at 148.59 171.45 0)
+    (property "LCSC" "C5369222" (at 148.59 171.45 0)
       (effects (font (size 1.27 1.27)) hide)
     )
@@
       (effects (font (size 1.27 1.27)) hide)
     )
-    (property "LCSC" "" (at 251.46 43.18 0)
+    (property "LCSC" "NotAvailable" (at 251.46 43.18 0)
       (effects (font (size 1.27 1.27)) hide)
     )
@@
       (effects (font (size 1.27 1.27)) hide)
     )
-    (property "LCSC" "" (at 86.36 52.07 0)
+    (property "LCSC" "NotAvailable" (at 86.36 52.07 0)
       (effects (font (size 1.27 1.27)) hide)
     )
@@
       (effects (font (size 1.27 1.27)) hide)
     )
-    (property "LCSC" "" (at 45.72 166.37 0)
+    (property "LCSC" "NotAvailable" (at 45.72 166.37 0)
       (effects (font (size 1.27 1.27)) hide)
     )
@@
       (effects (font (size 1.27 1.27)) hide)
     )
-    (property "LCSC" "" (at 243.84 109.22 0)
+    (property "LCSC" "NotAvailable" (at 243.84 109.22 0)
       (effects (font (size 1.27 1.27)) hide)
     )
@@
       (effects (font (size 1.27 1.27)) hide)
     )
-    (property "LCSC" "" (at 204.47 134.62 0)
+    (property "LCSC" "C849180" (at 204.47 134.62 0)
       (effects (font (size 1.27 1.27)) hide)
     )
@@
       (effects (font (size 1.27 1.27)) hide)
     )
-    (property "LCSC" "" (at 204.47 142.24 0)
+    (property "LCSC" "C844775" (at 204.47 142.24 0)
       (effects (font (size 1.27 1.27)) hide)
     )
@@
       (effects (font (size 1.27 1.27)) hide)
     )
-    (property "LCSC" "" (at 125.73 101.6 0)
+    (property "LCSC" "C844746" (at 125.73 101.6 0)
       (effects (font (size 1.27 1.27)) hide)
     )
@@
       (effects (font (size 1.27 1.27)) hide)
     )
-    (property "LCSC" "" (at 217.17 152.4 0)
+    (property "LCSC" "C185333" (at 217.17 152.4 0)
       (effects (font (size 1.27 1.27)) hide)
     )
@@
       (effects (font (size 1.27 1.27)) hide)
     )
-    (property "LCSC" "" (at 240.03 146.05 0)
+    (property "LCSC" "NotAvailable" (at 240.03 146.05 0)
       (effects (font (size 1.27 1.27)) hide)
     )
@@
       (effects (font (size 1.27 1.27)) hide)
     )
-    (property "LCSC" "" (at 161.29 133.35 0)
+    (property "LCSC" "C5369222" (at 161.29 133.35 0)
       (effects (font (size 1.27 1.27)) hide)
     )
@@
       (effects (font (size 1.27 1.27)) hide)
     )
-    (property "LCSC" "C105580" (at 151.13 133.35 0)
+    (property "LCSC" "C1854765" (at 151.13 133.35 0)
       (effects (font (size 1.27 1.27)) hide)
     )
@@
       (effects (font (size 1.27 1.27)) hide)
     )
-    (property "LCSC" "" (at 142.24 133.35 0)
+    (property "LCSC" "C5369222" (at 142.24 133.35 0)
       (effects (font (size 1.27 1.27)) hide)
     )
@@
       (effects (font (size 1.27 1.27)) hide)
     )
-    (property "LCSC" "" (at 130.81 133.35 0)
+    (property "LCSC" "C844180" (at 130.81 133.35 0)
       (effects (font (size 1.27 1.27)) hide)
     )
@@
       (effects (font (size 1.27 1.27)) hide)
     )
-    (property "LCSC" "" (at 265.43 91.44 0)
+    (property "LCSC" "C2883763" (at 265.43 91.44 0)
       (effects (font (size 1.27 1.27)) hide)
     )
@@
       (effects (font (size 1.27 1.27)) hide)
     )
-    (property "LCSC" "" (at 49.53 123.19 0)
+    (property "LCSC" "C844782" (at 49.53 123.19 0)
       (effects (font (size 1.27 1.27)) hide)
     )
@@
       (effects (font (size 1.27 1.27)) hide)
     )
-    (property "LCSC" "" (at 68.58 57.15 0)
+    (property "LCSC" "C246008" (at 68.58 57.15 0)
       (effects (font (size 1.27 1.27)) hide)
     )
@@
       (effects (font (size 1.27 1.27)) hide)
     )
-    (property "LCSC" "" (at 138.43 54.61 0)
+    (property "LCSC" "C2091473" (at 138.43 54.61 0)
       (effects (font (size 1.27 1.27)) hide)
     )
@@
       (effects (font (size 1.27 1.27)) hide)
     )
-    (property "LCSC" "" (at 128.27 186.69 0)
+    (property "LCSC" "C844180" (at 128.27 186.69 0)
       (effects (font (size 1.27 1.27)) hide)
     )
@@
       (effects (font (size 1.27 1.27)) hide)
     )
-    (property "LCSC" "" (at 233.68 45.72 0)
+    (property "LCSC" "C844782" (at 233.68 45.72 0)
       (effects (font (size 1.27 1.27)) hide)
     )
@@
       (effects (font (size 1.27 1.27)) hide)
     )
-    (property "LCSC" "" (at 82.55 62.23 0)
+    (property "LCSC" "C2992526" (at 82.55 62.23 0)
       (effects (font (size 1.27 1.27)) hide)
     )
@@
       (effects (font (size 1.27 1.27)) hide)
     )
-    (property "LCSC" "" (at 151.13 52.07 0)
+    (property "LCSC" "C2075334" (at 151.13 52.07 0)
       (effects (font (size 1.27 1.27)) hide)
     )
@@
       (effects (font (size 1.27 1.27)) hide)
     )
-    (property "LCSC" "" (at 149.86 34.29 0)
+    (property "LCSC" "C5369222" (at 149.86 34.29 0)
       (effects (font (size 1.27 1.27)) hide)
     )
@@
       (effects (font (size 1.27 1.27)) hide)
     )
-    (property "LCSC" "" (at 148.59 57.15 0)
+    (property "LCSC" "C2085910" (at 148.59 57.15 0)
       (effects (font (size 1.27 1.27)) hide)
     )
@@
       (effects (font (size 1.27 1.27)) hide)
     )
-    (property "LCSC" "" (at 223.52 50.8 0)
+    (property "LCSC" "C844773" (at 223.52 50.8 0)
       (effects (font (size 1.27 1.27)) hide)
     )
@@
       (effects (font (size 1.27 1.27)) hide)
     )
-    (property "LCSC" "" (at 59.69 31.75 0)
-      (effects (font (size 1.27 1.27)) hide)
-    )
+    (property "LCSC" "C2654002" (at 59.69 31.75 0)
+      (effects (font (size 1.27 1.27)) hide)
+    )
