File: mainboard-v05/RF_and_GPS.kicad_sch (KiCad schematic)
At the start: 23 parts, among them J12 Amphenol_901-144, J5 Amphenol_901-144, J6 Amphenol_901-144, J7 Amphenol_901-144, U10 XTB-40, U11 XTB-40, U12 XTB-40, U13 EP2W+, U14 S1216V8, U15 RFM9xBreakout, U20 RFM9xBreakout, U23 RFM98PW, U24 RFM98PW, U9 XTB-40

Commit message: Added more fields to BOM.
Parts:
- C44, C46: LCSC (none) -> C1691
- R24: LCSC (none) -> C1511834
Changed lines of the file:
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@@
       (effects (font (size 1.27 1.27)) hide)
     )
-    (property "LCSC" "" (at 240.03 109.22 0)
+    (property "LCSC" "C1511834" (at 240.03 109.22 0)
       (effects (font (size 1.27 1.27)) hide)
     )
@@
       (effects (font (size 1.27 1.27)) hide)
     )
-    (property "LCSC" "" (at 45.72 124.46 0)
+    (property "LCSC" "C1691" (at 45.72 124.46 0)
       (effects (font (size 1.27 1.27)) hide)
     )
@@
       (effects (font (size 1.27 1.27) bold))
     )
-    (property "LCSC" "" (at 125.73 124.46 0)
-      (effects (font (size 1.27 1.27)) hide)
-    )
+    (property "LCSC" "C1691" (at 125.73 124.46 0)
+      (effects (font (size 1.27 1.27)) hide)
+    )

Commit message: edits
Parts:
- R54, R56, R57, R58: LCSC (none) -> C1854765
- U23, U24: LCSC (none) -> NotAvailable

Commit message: Improved Py-Cubed BOM
Parts:
- J12, J5, J6, J7: LCSC (none) -> NotAvailable
- R43, R5: LCSC (none) -> C1511834
- R54, R56, R57, R58: LCSC C1854765 -> C3988417
Changed lines of the file:
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@@
       (effects (font (size 1.27 1.27)) hide)
     )
-    (property "LCSC" "" (at 256.54 59.69 0)
+    (property "LCSC" "NotAvailable" (at 256.54 59.69 0)
       (effects (font (size 1.27 1.27)) hide)
     )
@@
       (effects (font (size 1.27 1.27)) hide)
     )
-    (property "LCSC" "" (at 256.54 69.85 0)
+    (property "LCSC" "NotAvailable" (at 256.54 69.85 0)
       (effects (font (size 1.27 1.27)) hide)
     )
@@
       (effects (font (size 1.27 1.27)) hide)
     )
-    (property "LCSC" "" (at 78.74 129.54 0)
+    (property "LCSC" "NotAvailable" (at 78.74 129.54 0)
       (effects (font (size 1.27 1.27)) hide)
     )
@@
       (effects (font (size 1.27 1.27)) hide)
     )
-    (property "LCSC" "" (at 156.21 187.96 0)
+    (property "LCSC" "NotAvailable" (at 156.21 187.96 0)
       (effects (font (size 1.27 1.27)) hide)
     )
@@
       (effects (font (size 1.27 1.27)) hide)
     )
-    (property "LCSC" "" (at 102.87 134.62 0)
+    (property "LCSC" "C1511834" (at 102.87 134.62 0)
       (effects (font (size 1.27 1.27)) hide)
     )
@@
       (effects (font (size 1.27 1.27)) hide)
     )
-    (property "LCSC" "" (at 22.86 134.62 0)
+    (property "LCSC" "C1511834" (at 22.86 134.62 0)
       (effects (font (size 1.27 1.27)) hide)
     )
@@
       (effects (font (size 1.27 1.27)) hide)
     )
-    (property "LCSC" "C1854765" (at 139.7 62.23 0)
+    (property "LCSC" "C3988417" (at 139.7 62.23 0)
       (effects (font (size 1.27 1.27)) hide)
     )
@@
       (effects (font (size 1.27 1.27) bold) (justify left))
     )
-    (property "LCSC" "C1854765" (at 139.7 69.85 0)
+    (property "LCSC" "C3988417" (at 139.7 69.85 0)
       (effects (font (size 1.27 1.27)) hide)
     )
@@
       (effects (font (size 1.27 1.27)) hide)
     )
-    (property "LCSC" "C1854765" (at 77.47 62.23 0)
+    (property "LCSC" "C3988417" (at 77.47 62.23 0)
       (effects (font (size 1.27 1.27)) hide)
     )
@@
       (effects (font (size 1.27 1.27) bold) (justify left))
     )
-    (property "LCSC" "C1854765" (at 77.47 69.85 0)
-      (effects (font (size 1.27 1.27)) hide)
-    )
+    (property "LCSC" "C3988417" (at 77.47 69.85 0)
+      (effects (font (size 1.27 1.27)) hide)
+    )
