File: SidePanel/SidePanel.kicad_pcb (KiCad board)
At the start: 2 copper layers, 210 x 84 mm, 19 parts, among them J1 Conn_01x02_Pin

Commit message: SidePanel Rev1
Routing:
- net Net-(D1-A): track 82.5 -> 88.6 mm
- net /VN: track 183.9 -> 184.9 mm
