File: SidePanel/SidePanel.kicad_sch (KiCad schematic)
At the start: 19 parts, among them J1 Conn_01x02_Pin

Commit message: SidePanel Rev1
Parts:
- R1: now not fitted
Changed lines of the file:
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@@
 		(in_bom yes)
 		(on_board yes)
-		(dnp no)
+		(dnp yes)
 		(property "Reference" "R1"
 			(at 53.086 35.814 90)
